File: Remote Power Meter.kicad_pcb (KiCad board)
At the start: 2 copper layers, 110 x 45 mm, 25 parts, among them J1 USB_C_Receptacle_USB2.0, J2 USB_A, J3 Conn_01x04_Male, J4 Conn_01x04_Female, J5 Conn_01x02, J6 Conn_01x02, U1 AMS1117-3.3, U2 INA219AxD

Commit message: ...
Parts:
- added C4: 10nf, Capacitor_SMD:C_0603_1608Metric_Pad1.08x0.95mm_HandSolder, F.Cu at (71.0, 88.0)
- added C5: 100nf, Capacitor_SMD:C_0603_1608Metric_Pad1.08x0.95mm_HandSolder, F.Cu at (67.0, 78.0)
- added R10: 10K, Resistor_SMD:R_0603_1608Metric_Pad0.98x0.95mm_HandSolder, F.Cu at (78.0, 82.0)
- added R11: 10K, Resistor_SMD:R_0603_1608Metric_Pad0.98x0.95mm_HandSolder, F.Cu at (78.0, 84.0)
- added R12: 10K, Resistor_SMD:R_0603_1608Metric_Pad0.98x0.95mm_HandSolder, F.Cu at (121.9, 81.2)
- added SW1: SW_Push, Tinker:SW_Push_TS273014TP, F.Cu at (116.0, 82.0)
- added U3: CH340C, Package_SO:SOIC-16_3.9x9.9mm_P1.27mm, F.Cu at (70.0, 83.0)
- moved C1 21.1 mm to (52.0, 86.5), turned to 0 degrees
- moved U1 12.1 mm to (52.0, 80.4), turned to 180 degrees
Connections:
- J1 pad A6: unconnected-(J1-PadA6) -> UD+
- J1 pad A7: unconnected-(J1-PadA7) -> UD-
- J1 pad B6: unconnected-(J1-PadB6) -> UD+
- J1 pad B7: unconnected-(J1-PadB7) -> UD-
- Um1 pad 7: unconnected-(Um1-Pad7) -> TxD
- Um1 pad 8: unconnected-(Um1-Pad8) -> RxD
- Um1 pad 9: unconnected-(Um1-Pad9) -> RST
Routing:
- net RxD: track 0.00 -> 27.5 mm, vias 0 -> 2
- net TxD: track 0.00 -> 25.0 mm, vias 0 -> 2
- net UD-: track 0.00 -> 21.5 mm, vias 0 -> 2
- net UD+: track 0.00 -> 20.1 mm, vias 0 -> 2
- net RST: track 0.00 -> 16.3 mm
- net Net-(R11-Pad1): track 0.00 -> 11.8 mm
- net Net-(R10-Pad1): track 0.00 -> 11.2 mm
- net GND: track 22.4 -> 29.5 mm, vias 6 -> 10
- net Vcc: track 14.3 -> 16.5 mm
