File: Remote Power Meter.kicad_sch (KiCad schematic)
At the start: 23 parts, among them J1 USB_C_Receptacle_USB2.0, J2 USB_A, J3 Conn_01x04_Male, J4 Conn_01x04_Female, J5 Conn_01x02, J6 Conn_01x02, U1 AMS1117-3.3, U2 INA219AxD

Commit message: ...
Parts:
- added C4: 10nf, Capacitor_SMD:C_0603_1608Metric_Pad1.08x0.95mm_HandSolder, symbol Device:C
- added C5: 100nf, Capacitor_SMD:C_0603_1608Metric_Pad1.08x0.95mm_HandSolder, symbol Device:C
- added R10, R11, R12: 10K, Resistor_SMD:R_0603_1608Metric_Pad0.98x0.95mm_HandSolder, symbol Device:R
- added SW1: SW_Push, Tinker:SW_Push_TS273014TP, symbol Switch:SW_Push
- added U3: CH340C, Package_SO:SOIC-16_3.9x9.9mm_P1.27mm, symbol Interface_USB:CH340G
- renumbered J4 to J2, J5 to J4, J2 to J5
Connections:
- net 3v3: now also C4.1, C5.1, R12.1, U3.16 (VCC), U3.4 (V3)
- net GND: now also C4.2, C5.2, SW1.1, U3.1 (GND)
- net TxD: now reaches Um1.7 (GPIO1)
- net TxD: now also R11.2
- net RxD: now reaches Um1.8 (GPIO3)
- net RxD: now also R10.2
- net RST: now reaches Um1.9 (~{RST})
- net RST: now also R12.2, SW1.2
- net UD+: now reaches J1.A6 (D+)
- net UD+: now also J1.B6 (D+), U3.5 (UD+)
- net UD-: now reaches J1.A7 (D-)
- net UD-: now also J1.B7 (D-), U3.6 (UD-)
- new net: R10.1, U3.2 (TXD)
- new net: R11.1, U3.3 (RXD)
- new net CTS: U3.9 (~{CTS})
- new net DCD: U3.12 (~{DCD})
- new net DSR: U3.10 (~{DSR})
- new net DTR: U3.13 (~{DTR})
- new net RI: U3.11 (~{RI})
- new net RTS: U3.14 (~{RTS})
- no-connect marks 6 -> 17
Other:
- note added: "Can replace the CH340G with a CH340C & then leave off Y1, C3 & C4 (Actually done here...)"
- note added: "ESP Programmer"
- note added: "Programmer"
